Commit message: [FEAT]Calculations without square root operation

File: src/ros_ws/urdf_to_dh_package/install/urdf_to_dh/share/urdf_to_dh/urdf/ur5_mk2.urdf (robot description, URDF)
Before this commit: robot ur5_robot, 13 links, 12 joints
Joints:
- joint base_link-base_link_inertia: origin xyz=0 0 0 rpy=0 0 0 -> xyz=0 0 0 rpy=0 0 1.5707963267948966
- joint shoulder_lift_joint: limit lower=-3.141592653589793 upper=3.141592653589793 effort=150.0 velocity=3.141592653589793 -> lower=-6.283185307179586 upper=6.283185307179586 effort=150.0 velocity=3.141592653589793
- joint shoulder_pan_joint: limit lower=-3.141592653589793 upper=3.141592653589793 effort=150.0 velocity=3.141592653589793 -> lower=-6.283185307179586 upper=6.283185307179586 effort=150.0 velocity=3.141592653589793
- joint wrist_1_joint: limit lower=-3.141592653589793 upper=3.141592653589793 effort=28.0 velocity=3.141592653589793 -> lower=-6.283185307179586 upper=6.283185307179586 effort=28.0 velocity=3.141592653589793
- joint wrist_2_joint: limit lower=-3.141592653589793 upper=3.141592653589793 effort=28.0 velocity=3.141592653589793 -> lower=-6.283185307179586 upper=6.283185307179586 effort=28.0 velocity=3.141592653589793
- joint wrist_3_joint: limit lower=-3.141592653589793 upper=3.141592653589793 effort=28.0 velocity=3.141592653589793 -> lower=-6.283185307179586 upper=6.283185307179586 effort=28.0 velocity=3.141592653589793

File: src/ros_ws/urdf_to_dh_package/urdf/ur5_calib.urdf (robot description, URDF)
Before this commit: robot ur5_robot, 13 links, 12 joints
Joints:
- joint base_link-base_link_inertia: origin xyz=0 0 0 rpy=0 0 0 -> xyz=0 0 0 rpy=0 0 1.5707963267948966
- joint shoulder_lift_joint: limit lower=-3.141592653589793 upper=3.141592653589793 effort=150.0 velocity=3.141592653589793 -> lower=-6.283185307179586 upper=6.283185307179586 effort=150.0 velocity=3.141592653589793
- joint shoulder_pan_joint: limit lower=-3.141592653589793 upper=3.141592653589793 effort=150.0 velocity=3.141592653589793 -> lower=-6.283185307179586 upper=6.283185307179586 effort=150.0 velocity=3.141592653589793
- joint wrist_1_joint: limit lower=-3.141592653589793 upper=3.141592653589793 effort=28.0 velocity=3.141592653589793 -> lower=-6.283185307179586 upper=6.283185307179586 effort=28.0 velocity=3.141592653589793
- joint wrist_2_joint: limit lower=-3.141592653589793 upper=3.141592653589793 effort=28.0 velocity=3.141592653589793 -> lower=-6.283185307179586 upper=6.283185307179586 effort=28.0 velocity=3.141592653589793
- joint wrist_3_joint: limit lower=-3.141592653589793 upper=3.141592653589793 effort=28.0 velocity=3.141592653589793 -> lower=-6.283185307179586 upper=6.283185307179586 effort=28.0 velocity=3.141592653589793

File: src/ros_ws/urdf_to_dh_package/urdf/ur5_kin_modified.urdf (robot description, URDF)
Before this commit: robot ur5_robot, 13 links, 12 joints
Joints:
- joint base_link-base_link_inertia: origin xyz=0 0 0 rpy=0 0 0 -> xyz=0 0 0 rpy=0 0 1.5707963267948966
- joint elbow_joint: origin xyz=-0.425 0 0 rpy=0 0 0 -> xyz=-0.39225 0 0 rpy=0 0 0
- joint shoulder_lift_joint: limit lower=-3.141592653589793 upper=3.141592653589793 effort=150.0 velocity=3.141592653589793 -> lower=-6.283185307179586 upper=6.283185307179586 effort=150.0 velocity=3.141592653589793; origin xyz=0 0 0 rpy=1.570796327 0 0 -> xyz=-0.425 0 0 rpy=0 0 0
- joint shoulder_pan_joint: limit lower=-3.141592653589793 upper=3.141592653589793 effort=150.0 velocity=3.141592653589793 -> lower=-6.283185307179586 upper=6.283185307179586 effort=150.0 velocity=3.141592653589793; origin xyz=0 0 0.089159 rpy=0 0 0 -> xyz=0 0 0.089159 rpy=1.570796327 0 0
- joint wrist_1_joint: limit lower=-3.141592653589793 upper=3.141592653589793 effort=28.0 velocity=3.141592653589793 -> lower=-6.283185307179586 upper=6.283185307179586 effort=28.0 velocity=3.141592653589793; origin xyz=-0.39225 0 0.10915 rpy=0 0 0 -> xyz=0 0 0.10915 rpy=1.570796327 0 0
- joint wrist_2_joint: limit lower=-3.141592653589793 upper=3.141592653589793 effort=28.0 velocity=3.141592653589793 -> lower=-6.283185307179586 upper=6.283185307179586 effort=28.0 velocity=3.141592653589793; origin xyz=0 -0.09465 -1.941303950897609e-11 rpy=1.570796327 0 0 -> xyz=0 0 0.09465 rpy=-1.570796327 0 0
- joint wrist_3_joint: limit lower=-3.141592653589793 upper=3.141592653589793 effort=28.0 velocity=3.141592653589793 -> lower=-6.283185307179586 upper=6.283185307179586 effort=28.0 velocity=3.141592653589793; origin xyz=0 0.0823 -1.688001216681175e-11 rpy=1.570796326589793 3.141592653589793 3.141592653589793 -> xyz=0 0 0.0823 rpy=0 0 0
